File: ARM-Cortex_M0.brd (EAGLE design)
At the start: 50 x 50 mm, 9 parts, among them IC1 SAMD21G18A-AUT, J2 CORTEX_DEBUGPTH, Y3 32,768Khz_SMD

Commit message: hardware
hardware
Parts:
- added C7: 1uF, KarlVaello-Capacitors:C0603
- added J1, J10, J3, J4, J5, J6, J7, J8, J9: (no value), SparkFun-Connectors:1X01NS-KIT
- added J11: (no value), SparkFun-Connectors:USB-B-MICRO-SMD_V03
- added U1: MIC5203-3.3, SparkFun-PowerIC:SOT23-5
- moved C6 21.9 mm to (24.7, 33.1), turned to 270 degrees
- moved J2 20.4 mm to (8.50, 27.1), turned to 90 degrees
Connections:
- new net RAW: U1.1, U1.3
- net +3V3: now also C7.2, U1.5
- net GND: now also C7.1, U1.2
Changed lines of the file:
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@@
 <?xml version="1.0" encoding="utf-8"?>
 <!DOCTYPE eagle SYSTEM "eagle.dtd">
-<eagle version="7.4.0">
+<eagle version="7.7.0">
 <drawing>
 <settings>
@@
 <element name="C4" library="KarlVaello-Capacitors" package="C0603" value="" x="24.3" y="16.9" rot="R270"/>
 <element name="C5" library="KarlVaello-Capacitors" package="C0603" value="100nF" x="21.5" y="16.5" rot="R90"/>
-<element name="J2" library="SparkFun-Connectors" package="2X5-PTH-1.27MM" value="CORTEX_DEBUGPTH" x="7" y="6.8"/>
-<element name="C6" library="KarlVaello-Capacitors" package="C0603" value="1uF" x="11.2" y="15.8"/>
+<element name="J2" library="SparkFun-Connectors" package="2X5-PTH-1.27MM" value="CORTEX_DEBUGPTH" x="8.5" y="27.1" rot="R90"/>
+<element name="C6" library="KarlVaello-Capacitors" package="C0603" value="1uF" x="24.7" y="33.1" rot="R270"/>
+<element name="U1" library="SparkFun-PowerIC" package="SOT23-5" value="MIC5203-3.3" x="12.9" y="17">
+<attribute name="PROD_ID" value="VREG-00822" x="12.9" y="17" size="1.778" layer="27" display="off"/>
+</element>
+<element name="C7" library="KarlVaello-Capacitors" package="C0603" value="1uF" x="8.3" y="22.5"/>
+<element name="J1" library="SparkFun-Connectors" package="1X01NS-KIT" value="" x="2.9" y="20.8"/>
+<element name="J3" library="SparkFun-Connectors" package="1X01NS-KIT" value="" x="2.9" y="18.7"/>
+<element name="J4" library="SparkFun-Connectors" package="1X01NS-KIT" value="" x="2.9" y="16.6"/>
+<element name="J5" library="SparkFun-Connectors" package="1X01NS-KIT" value="" x="2.9" y="14.5"/>
+<element name="J6" library="SparkFun-Connectors" package="1X01NS-KIT" value="" x="2.9" y="12.4"/>
+<element name="J7" library="SparkFun-Connectors" package="1X01NS-KIT" value="" x="2.9" y="10.3"/>
+<element name="J8" library="SparkFun-Connectors" package="1X01NS-KIT" value="" x="2.9" y="8.2"/>
+<element name="J9" library="SparkFun-Connectors" package="1X01NS-KIT" value="" x="2.9" y="6.1"/>
+<element name="J10" library="SparkFun-Connectors" package="1X01NS-KIT" value="" x="2.9" y="4"/>
+<element name="J11" library="SparkFun-Connectors" package="USB-B-MICRO-SMD_V03" value="" x="29.9" y="2" rot="R90">
+<attribute name="PROD_ID" value="CONN-11752" x="29.9" y="2" size="1.778" layer="27" rot="R90" display="off"/>
+</element>
 </elements>
 <signals>
@@
 <contactref element="J2" pad="5"/>
 <contactref element="C6" pad="1"/>
+<contactref element="U1" pad="2"/>
+<contactref element="C7" pad="1"/>
 <wire x1="27.5" y1="27.25" x2="25.25" y2="29.275" width="0" layer="19" extent="1-1"/>
 </signal>
@@
 <contactref element="C5" pad="2"/>
 <contactref element="J2" pad="1"/>
+<contactref element="U1" pad="5"/>
+<contactref element="C7" pad="2"/>
 <wire x1="29.275" y1="27.75" x2="32.15" y2="27.8" width="0" layer="19" extent="1-1"/>
 <wire x1="24.25" y1="29.275" x2="29.275" y2="27.75" width="0" layer="19" extent="1-1"/>
@@
 <wire x1="24.3" y1="17.75" x2="24.25" y2="20.725" width="0" layer="19" extent="1-1"/>
 <wire x1="21.5" y1="17.35" x2="24.3" y2="17.75" width="0" layer="19" extent="1-1"/>
-<wire x1="4.46" y1="6.165" x2="21.5" y2="17.35" width="0" layer="19" extent="1-1"/>
+<wire x1="11.95" y1="18.3001" x2="21.5" y2="17.35" width="0" layer="19" extent="1-1"/>
+<wire x1="9.15" y1="22.5" x2="11.95" y2="18.3001" width="0" layer="19" extent="1-1"/>
+<wire x1="9.135" y1="24.56" x2="9.15" y2="22.5" width="0" layer="19" extent="1-1"/>
 </signal>
 <signal name="N$5">
@@
 <contactref element="IC1" pad="43"/>
 <contactref element="C6" pad="2"/>
-<wire x1="12.05" y1="15.8" x2="24.75" y2="29.275" width="0" layer="19" extent="1-1"/>
+<wire x1="24.75" y1="29.275" x2="24.7" y2="32.25" width="0" layer="19" extent="1-1"/>
+</signal>
+<signal name="RAW">
+<contactref element="U1" pad="1"/>
+<contactref element="U1" pad="3"/>
+<wire x1="11.95" y1="15.6999" x2="13.85" y2="15.6999" width="0" layer="19" extent="1-1"/>
 </signal>
 </signals>

Commit message: Eagle file version update
from 7.5.0 to 7.7.0
Parts:
- moved J11 4.30 mm to (30.0, 6.30)
Changed lines of the file:
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@@
 <element name="J9" library="SparkFun-Connectors" package="1X01NS-KIT" value="" x="2.9" y="6.1"/>
 <element name="J10" library="SparkFun-Connectors" package="1X01NS-KIT" value="" x="2.9" y="4"/>
-<element name="J11" library="SparkFun-Connectors" package="USB-B-MICRO-SMD_V03" value="" x="29.9" y="2" rot="R90">
-<attribute name="PROD_ID" value="CONN-11752" x="29.9" y="2" size="1.778" layer="27" rot="R90" display="off"/>
+<element name="J11" library="SparkFun-Connectors" package="USB-B-MICRO-SMD_V03" value="" x="30" y="6.3" rot="R90">
+<attribute name="PROD_ID" value="CONN-11752" x="30" y="6.3" size="1.778" layer="27" rot="R90" display="off"/>
 </element>
 </elements>

Commit message: Hardware modifications
Hardware modifications
Parts:
- added C8: 10nF, KarlVaello-Capacitors:C0603
- added R1: 330R, KarlVaello-Resistors:R0603
- added R2: 10K, KarlVaello-Resistors:R0603
- added S1: SW-MOME, SparkFun-Electromechanical:TACTILE-SWITCH-SMD
- added X1: MINI-USB_SHIELD4P-32005-101, con-cypressindustries:32005-101
- moved J11 26.0 mm to (48.0, 25.0), turned to 180 degrees
- moved C3 0.81 mm to (33.1, 28.6)
Connections:
- removed net N$3: IC1.46
- removed net N$4: IC1.45
- removed net N$5: J2.2
- removed net N$6: J2.4
- new net D0: IC1.16
- new net D1: IC1.15
- new net D10: IC1.27
- new net D11: IC1.25
- new net D12: IC1.28
- new net D13: IC1.26
- new net D2: IC1.23
- new net D3: IC1.14
- new net D4: IC1.13
- new net D5: IC1.24
- new net D6: IC1.29
- new net D7: IC1.30
- new net D8: IC1.11
- new net D9: IC1.12
- new net SWDCLK: IC1.45, J2.4
- new net SWDIO: IC1.46, J2.2
- new net TARGET_USB_N: IC1.33, J11.D-
- new net TARGET_USB_P: IC1.34, J11.D+
- new net TARGE_RESET: C8.2, IC1.40, R1.1
- new net VBUS: J11.VBUS
- net +3V3: now also R2.2
- net GND: now also C8.1, J11.GND, J11.SHIELD1, J11.SHIELD2, J11.SHIELD3, S1.3
- net RESET: now also R1.2, R2.1, S1.1
Routing:
- net TARGET_USB_N: track 0.00 -> 16.8 mm
- net TARGET_USB_P: track 0.00 -> 16.7 mm
Changed lines of the file:
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@@
 <element name="C1" library="KarlVaello-Capacitors" package="C0603" value="22pF" x="14" y="25.5" rot="R270"/>
 <element name="C2" library="KarlVaello-Capacitors" package="C0603" value="22pF" x="14" y="29.5" rot="R90"/>
-<element name="C3" library="KarlVaello-Capacitors" package="C0603" value="100nF" x="33" y="27.8" rot="R180"/>
+<element name="C3" library="KarlVaello-Capacitors" package="C0603" value="100nF" x="33.1" y="28.6" rot="R180"/>
 <element name="C4" library="KarlVaello-Capacitors" package="C0603" value="" x="24.3" y="16.9" rot="R270"/>
 <element name="C5" library="KarlVaello-Capacitors" package="C0603" value="100nF" x="21.5" y="16.5" rot="R90"/>
@@
 <element name="J9" library="SparkFun-Connectors" package="1X01NS-KIT" value="" x="2.9" y="6.1"/>
 <element name="J10" library="SparkFun-Connectors" package="1X01NS-KIT" value="" x="2.9" y="4"/>
-<element name="J11" library="SparkFun-Connectors" package="USB-B-MICRO-SMD_V03" value="" x="30" y="6.3" rot="R90">
-<attribute name="PROD_ID" value="CONN-11752" x="30" y="6.3" size="1.778" layer="27" rot="R90" display="off"/>
-</element>
+<element name="J11" library="SparkFun-Connectors" package="USB-B-MICRO-SMD_V03" value="" x="48" y="25" rot="R180">
+<attribute name="PROD_ID" value="CONN-11752" x="48" y="25" size="1.778" layer="27" rot="R180" display="off"/>
+</element>
+<element name="X1" library="con-cypressindustries" package="32005-101" value="MINI-USB_SHIELD4P-32005-101" x="46.5" y="13.9" rot="R180">
+<attribute name="OC_NEWARK" value="unknown" x="46.5" y="13.9" size="1.778" layer="27" rot="R180" display="off"/>
+<attribute name="OC_FARNELL" value="unknown" x="46.5" y="13.9" size="1.778" layer="27" rot="R180" display="off"/>
+<attribute name="MPN" value="" x="46.5" y="13.9" size="1.778" layer="27" rot="R180" display="off"/>
+<attribute name="MF" value="" x="46.5" y="13.9" size="1.778" layer="27" rot="R180" display="off"/>
+</element>
+<element name="S1" library="SparkFun-Electromechanical" package="TACTILE-SWITCH-SMD" value="SW-MOME" x="42.8" y="4.1">
+<attribute name="PROD_ID" value="SWCH-08247" x="42.8" y="4.1" size="1.778" layer="27" display="off"/>
+</element>
+<element name="C8" library="KarlVaello-Capacitors" package="C0603" value="10nF" x="21.3" y="11.6" rot="R270"/>
+<element name="R1" library="KarlVaello-Resistors" package="R0603" value="330R" x="18.2" y="11.9" rot="R90"/>
+<element name="R2" library="KarlVaello-Resistors" package="R0603" value="10K" x="18.8" y="16.6" rot="R90"/>
 </elements>
 <signals>
@@
 <contactref element="U1" pad="2"/>
 <contactref element="C7" pad="1"/>
+<contactref element="J11" pad="GND"/>
+<contactref element="J11" pad="SHIELD1"/>
+<contactref element="J11" pad="SHIELD3"/>
+<contactref element="J11" pad="SHIELD2"/>
+<contactref element="S1" pad="3"/>
+<contactref element="C8" pad="1"/>
 <wire x1="27.5" y1="27.25" x2="25.25" y2="29.275" width="0" layer="19" extent="1-1"/>
 </signal>
 <signal name="+3V3">
-<contactref element="IC1" pad="17"/>
-<contactref element="C3" pad="2"/>
 <contactref element="IC1" pad="36"/>
 <contactref element="C4" pad="1"/>
@@
 <contactref element="U1" pad="5"/>
 <contactref element="C7" pad="2"/>
-<wire x1="29.275" y1="27.75" x2="32.15" y2="27.8" width="0" layer="19" extent="1-1"/>
+<contactref element="IC1" pad="17"/>
+<contactref element="C3" pad="2"/>
+<contactref element="R2" pad="2"/>
+<wire x1="29.275" y1="27.75" x2="32.25" y2="28.6" width="0" layer="19" extent="1-1"/>
 <wire x1="24.25" y1="29.275" x2="29.275" y2="27.75" width="0" layer="19" extent="1-1"/>
 <wire x1="24.25" y1="20.725" x2="24.25" y2="29.275" width="0" layer="19" extent="1-1"/>
 <wire x1="24.3" y1="17.75" x2="24.25" y2="20.725" width="0" layer="19" extent="1-1"/>
 <wire x1="21.5" y1="17.35" x2="24.3" y2="17.75" width="0" layer="19" extent="1-1"/>
-<wire x1="11.95" y1="18.3001" x2="21.5" y2="17.35" width="0" layer="19" extent="1-1"/>
+<wire x1="18.8" y1="17.45" x2="21.5" y2="17.35" width="0" layer="19" extent="1-1"/>
+<wire x1="11.95" y1="18.3001" x2="18.8" y2="17.45" width="0" layer="19" extent="1-1"/>
 <wire x1="9.15" y1="22.5" x2="11.95" y2="18.3001" width="0" layer="19" extent="1-1"/>
 <wire x1="9.135" y1="24.56" x2="9.15" y2="22.5" width="0" layer="19" extent="1-1"/>
 </signal>
-<signal name="N$5">
+<signal name="SWDIO">
 <contactref element="J2" pad="2"/>
-</signal>
-<signal name="N$6">
+<contactref element="IC1" pad="46"/>
+<wire x1="7.865" y1="24.56" x2="23.25" y2="29.275" width="0" layer="19" extent="1-1"/>
+</signal>
+<signal name="SWDCLK">
 <contactref element="J2" pad="4"/>
+<contactref element="IC1" pad="45"/>
+<wire x1="7.865" y1="25.83" x2="23.75" y2="29.275" width="0" layer="19" extent="1-1"/>
 </signal>
 <signal name="RESET">
 <contactref element="J2" pad="10"/>
-</signal>
-<signal name="N$3">
-<contactref element="IC1" pad="46"/>
-</signal>
-<signal name="N$4">
-<contactref element="IC1" pad="45"/>
+<contactref element="R1" pad="2"/>
+<contactref element="R2" pad="1"/>
+<contactref element="S1" pad="1"/>
+<wire x1="18.2" y1="12.75" x2="40.006" y2="6.005" width="0" layer="19" extent="1-1"/>
+<wire x1="18.8" y1="15.75" x2="18.2" y2="12.75" width="0" layer="19" extent="1-1"/>
+<wire x1="7.865" y1="29.64" x2="18.8" y2="15.75" width="0" layer="19" extent="1-1"/>
 </signal>
 <signal name="N$7">
@@
 <wire x1="11.95" y1="15.6999" x2="13.85" y2="15.6999" width="0" layer="19" extent="1-1"/>
 </signal>
+<signal name="VBUS">
+<contactref element="J11" pad="VBUS"/>
+</signal>
+<signal name="TARGET_USB_N">
+<contactref element="J11" pad="D-"/>
+<contactref element="IC1" pad="33"/>
+<wire x1="29.275" y1="26.25" x2="40.25" y2="26.25" width="0.1524" layer="1"/>
+<wire x1="40.25" y1="26.25" x2="42.15" y2="24.35" width="0.1524" layer="1"/>
+<wire x1="42.15" y1="24.35" x2="45.275" y2="24.35" width="0.1524" layer="1"/>
+</signal>
+<signal name="TARGET_USB_P">
+<contactref element="J11" pad="D+"/>
+<contactref element="IC1" pad="34"/>
+<wire x1="29.275" y1="26.75" x2="40.55" y2="26.75" width="0.1524" layer="1"/>
+<wire x1="40.55" y1="26.75" x2="42.3" y2="25" width="0.1524" layer="1"/>
+<wire x1="42.3" y1="25" x2="45.275" y2="25" width="0.1524" layer="1"/>
+</signal>
+<signal name="TARGE_RESET">
+<contactref element="IC1" pad="40"/>
+<contactref element="C8" pad="2"/>
+<contactref element="R1" pad="1"/>
+<wire x1="21.3" y1="10.75" x2="26.25" y2="29.275" width="0" layer="19" extent="1-1"/>
+<wire x1="18.2" y1="11.05" x2="21.3" y2="10.75" width="0" layer="19" extent="1-1"/>
+</signal>
+<signal name="D13">
+<contactref element="IC1" pad="26"/>
+</signal>
+<signal name="D12">
+<contactref element="IC1" pad="28"/>
+</signal>
+<signal name="D11">
+<contactref element="IC1" pad="25"/>
+</signal>
+<signal name="D10">
+<contactref element="IC1" pad="27"/>
+</signal>
+<signal name="D9">
+<contactref element="IC1" pad="12"/>
+</signal>
+<signal name="D8">
+<contactref element="IC1" pad="11"/>
+</signal>
+<signal name="D7">
+<contactref element="IC1" pad="30"/>
+</signal>
+<signal name="D6">
+<contactref element="IC1" pad="29"/>
+</signal>
+<signal name="D5">
+<contactref element="IC1" pad="24"/>
+</signal>
+<signal name="D4">
+<contactref element="IC1" pad="13"/>
+</signal>
+<signal name="D3">
+<contactref element="IC1" pad="14"/>
+</signal>
+<signal name="D2">
+<contactref element="IC1" pad="23"/>
+</signal>
+<signal name="D1">
+<contactref element="IC1" pad="15"/>
+</signal>
+<signal name="D0">
+<contactref element="IC1" pad="16"/>
+</signal>
 </signals>
