File: ARM-Cortex_M0.sch (EAGLE design)
At the start: 21 parts, among them IC1 SAMD21G18A-AUT, J2 CORTEX_DEBUGPTH, U1 MIC5203-3.3, Y3 32,768Khz_SMD

Commit message: Hardware modifications
Hardware modifications
Parts:
- added C8: 10nF, KarlVaello-Capacitors:C-EUC0603
- added R1: 330R, KarlVaello-Resistors:R-EU_R0603
- added R2: 10K, KarlVaello-Resistors:R-EU_R0603
- added S1: SW-MOME, SparkFun-Electromechanical:SWITCH-MOMENTARY-2SMD
- added X1: MINI-USB_SHIELD4P-32005-101, con-cypressindustries:MINI-USB_SHIELD4P-32005-101
Connections:
- removed net N$3: IC1.PA31/EIC/SCOM1PAD3/TC1
- removed net N$4: IC1.PA30/EIC/SCOM1PAD2/TC1
- removed net N$5: J2.SWDIO/TMS
- removed net N$6: J2.SWDCLK/TCK
- new net D0: IC1.PA11/EIC/AIN19/SCOM2PAD3+/TC1
- new net D1: IC1.PA10/EIC/AIN18/SCOM2PAD2+/TC1
- new net D10: IC1.PA18/EIC/SCOM1PAD2+/TC3
- new net D11: IC1.PA16/I2C/EIC/SCOM1PAD0+/TC2
- new net D12: IC1.PA19/EIC/SCOM1PAD3+/TC3
- new net D13: IC1.PA17/I2C/EIC/SCOM1PAD1+/TC2
- new net D2: IC1.PA14/XIN/EIC/SCOM2PAD2+/TC3
- new net D3: IC1.PA9/I2C/EIC/AIN17/SCOM2PAD1+/TC0
- new net D4: IC1.PA8/I2C/AIN16/SCOM2PAD0+/TC0
- new net D5: IC1.PA15/XOUT/EIC/SCOM2PAD3+/TC3
- new net D6: IC1.PA20/EIC/SCOM5PAD2+
- new net D7: IC1.PA21/EIC/SCOM5PAD3+
- new net D8: IC1.PA6/EIC/AIN6/SCOM0PAD2/TC1
- new net D9: IC1.PA7/EIC/AIN7/SCOM0PAD3/TC1
- new net SWDCLK: IC1.PA30/EIC/SCOM1PAD2/TC1, J2.SWDCLK/TCK
- new net SWDIO: IC1.PA31/EIC/SCOM1PAD3/TC1, J2.SWDIO/TMS
- new net TARGET_USB_N: IC1.PA24/EIC/SCOM3PAD2+/TC5, J11.D-
- new net TARGET_USB_P: IC1.PA25/EIC/SCOM3PAD3+/TC5, J11.D+
- new net TARGE_RESET: C8.2, IC1.RESETN, R1.1
- new net VBUS: J11.VCC
- net +3V3: now also R2.2
- net GND: now also C8.1, J11.GND, J11.SHIELD, S1.2
- net RESET: now also R1.2, R2.1, S1.1
Other:
- note added: "ATSAMD21 MICROCONTROLLER"
- note added: "POWER AND FILTERING"
- note removed: "Micro"
- note removed: "POWER"
- moved on the sheet: C3, J11, J2

Commit message: hardware modifications
hardware modifications
Parts:
- removed J11: (no value), SparkFun-Connectors:USB_MICROB_PLUGCONN-11752
- removed X1: MINI-USB_SHIELD4P-32005-101, con-cypressindustries:MINI-USB_SHIELD4P-32005-101
- added J13: USB-MICROB", KarlVaello-Connectors:USB-MICROB"
Connections:
- net GND: now also J13.GND, J13.SHIELD; no longer J11.GND, J11.SHIELD
- net TARGET_USB_N: now also J13.D-; no longer J11.D-
- net TARGET_USB_P: now also J13.D+; no longer J11.D+
- net VBUS: now also J13.VBUS; no longer J11.VCC
Changed lines of the file:
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@@
 <part name="J9" library="SparkFun-Connectors" deviceset="M01" device="NOSILK-KIT"/>
 <part name="J10" library="SparkFun-Connectors" deviceset="M01" device="NOSILK-KIT"/>
-<part name="J11" library="SparkFun-Connectors" deviceset="USB_MICROB_PLUG" device="CONN-11752"/>
 <part name="GND11" library="KarlVaello-Simbols" deviceset="GND" device=""/>
 <part name="GND12" library="KarlVaello-Simbols" deviceset="GND" device=""/>
-<part name="X1" library="con-cypressindustries" deviceset="MINI-USB_SHIELD4P-" device="32005-101"/>
 <part name="S1" library="SparkFun-Electromechanical" deviceset="SWITCH-MOMENTARY-2" device="SMD" value="SW-MOME"/>
 <part name="GND13" library="KarlVaello-Simbols" deviceset="GND" device=""/>
@@
 <part name="R2" library="KarlVaello-Resistors" deviceset="R-EU_" device="R0603" value="10K"/>
 <part name="+3V1" library="KarlVaello-Simbols" deviceset="+3V3" device=""/>
+<part name="J13" library="KarlVaello-Connectors" deviceset="USB-MICROB" device="&quot;"/>
 </parts>
 <sheets>
@@
 <instance part="J9" gate="G$1" x="205.74" y="30.48"/>
 <instance part="J10" gate="G$1" x="205.74" y="43.18"/>
-<instance part="J11" gate="G$1" x="50.8" y="96.52"/>
-<instance part="GND11" gate="1" x="68.58" y="93.98"/>
+<instance part="GND11" gate="1" x="58.42" y="104.14"/>
 <instance part="GND12" gate="1" x="40.64" y="88.9"/>
-<instance part="X1" gate="G$1" x="58.42" y="116.84"/>
 <instance part="S1" gate="G$1" x="106.68" y="55.88" rot="R270"/>
 <instance part="GND13" gate="1" x="106.68" y="45.72"/>
@@
 <instance part="R2" gate="G$1" x="106.68" y="71.12" rot="R90"/>
 <instance part="+3V1" gate="G$1" x="106.68" y="81.28"/>
+<instance part="J13" gate="G$1" x="48.26" y="99.06" rot="MR180"/>
 </instances>
 <busses>
@@
 </segment>
 <segment>
-<pinref part="J11" gate="G$1" pin="GND"/>
 <pinref part="GND12" gate="1" pin="GND"/>
 <wire x1="40.64" y1="91.44" x2="43.18" y2="91.44" width="0.1524" layer="91"/>
-</segment>
-<segment>
-<pinref part="J11" gate="G$1" pin="SHIELD"/>
+<pinref part="J13" gate="G$1" pin="GND"/>
+</segment>
+<segment>
 <pinref part="GND11" gate="1" pin="GND"/>
-<wire x1="68.58" y1="96.52" x2="58.42" y2="96.52" width="0.1524" layer="91"/>
+<pinref part="J13" gate="G$1" pin="SHIELD"/>
+<wire x1="43.18" y1="104.14" x2="43.18" y2="106.68" width="0.1524" layer="91"/>
+<wire x1="43.18" y1="106.68" x2="58.42" y2="106.68" width="0.1524" layer="91"/>
 </segment>
 <segment>
@@
 <net name="VBUS" class="0">
 <segment>
-<pinref part="J11" gate="G$1" pin="VCC"/>
 <wire x1="43.18" y1="101.6" x2="22.86" y2="101.6" width="0.1524" layer="91"/>
 <label x="22.86" y="101.6" size="1.27" layer="95" font="vector" rot="R180" xref="yes"/>
+<pinref part="J13" gate="G$1" pin="VBUS"/>
 </segment>
 </net>
 <net name="TARGET_USB_N" class="0">
 <segment>
-<pinref part="J11" gate="G$1" pin="D-"/>
 <wire x1="43.18" y1="99.06" x2="22.86" y2="99.06" width="0.1524" layer="91"/>
 <label x="22.86" y="99.06" size="1.27" layer="95" font="vector" rot="R180" xref="yes"/>
+<pinref part="J13" gate="G$1" pin="D-"/>
 </segment>
 <segment>
@@
 <net name="TARGET_USB_P" class="0">
 <segment>
-<pinref part="J11" gate="G$1" pin="D+"/>
 <wire x1="43.18" y1="96.52" x2="22.86" y2="96.52" width="0.1524" layer="91"/>
 <label x="22.86" y="96.52" size="1.27" layer="95" font="vector" rot="R180" xref="yes"/>
-</segment>
-<segment>
+<pinref part="J13" gate="G$1" pin="D+"/>
+</segment>
+<segment>

Commit message: Hardaware modification, programing ARM info
Hardaware modification, programing ARM info
Parts:
- removed C3: 100nF, KarlVaello-Capacitors:C-EUC0603
- removed C4: (no value), KarlVaello-Capacitors:C-EUC0603
- removed J10, J5, J6, J7, J8, J9: (no value), SparkFun-Connectors:M01NOSILK-KIT
- added C10: 10uF, KarlVaello-Capacitors:C-EUC0603
- added C9: 1uF, KarlVaello-Capacitors:C-EUC0603
- added D1, D5: GREEN, SparkFun-LED:LED0603
- added D2: YELLOW, SparkFun-LED:LED0603
- added D3: MBR120, diode:CGRM4001-G
- added D4: ORANGE, SparkFun-LED:LED0603
- added J21: (no value), SparkFun-Connectors:JST_2MM_MALE
- added J28: (no value), SparkFun-Connectors:M15
- added R3: 100K, KarlVaello-Resistors:R-EU_R0603
- added R4, R5: 1K, KarlVaello-Resistors:R-EU_R0603
- C5: value 100nF -> 10uF
- C8: value 10nF -> 10uF
- J1: device SparkFun-Connectors:M01NOSILK-KIT -> SparkFun-Connectors:M15
- J3, J4: device SparkFun-Connectors:M01NOSILK-KIT -> SparkFun-Connectors:M04NO_SILK_ALL_ROUND
- R1: value 330R -> 1K
- R2: value 10K -> 1K
- U1: value MIC5203-3.3 -> SPX3918-3.3; device SparkFun-PowerIC:MIC52053.3V -> SparkFun-PowerIC:V_REG_AP2112K-3.3V
Connections:
- removed net D0: IC1.PA11/EIC/AIN19/SCOM2PAD3+/TC1
- removed net D1: IC1.PA10/EIC/AIN18/SCOM2PAD2+/TC1
- removed net RAW: U1.EN, U1.IN
- removed net TARGE_RESET: C8.2, IC1.RESETN, R1.1
- new net A0: IC1.PA2/EIC/AIN0, J28.11
- new net A1: IC1.PB8/EIC/AIN2/SCOM4PAD0/TC4, J28.10
- new net A2: IC1.PB9/EIC/AIN3/SCOM4PAD1//TC4, J28.9
- new net A3: IC1.PA4/EIC/REF/AIN4/SCOM0PAD0/TC0, J28.8
- new net A4: IC1.PA5/EIC/AIN5/SCOM0PAD1/TC0, J28.7
- new net A5: IC1.PB2/EIC/AIN10/SCOM5PAD0, J28.6
- new net AREF: C9.2, IC1.PA3/EIC/REF/AIN1, J28.13
- new net D0/RX: IC1.PA11/EIC/AIN19/SCOM2PAD3+/TC1, J1.4
- new net D1/TX: IC1.PA10/EIC/AIN18/SCOM2PAD2+/TC1, J1.3
- new net MISO: IC1.PA12/I2C/EIC/SCOM2PAD0+/TC2, J28.2
- new net MOSI: IC1.PB10/EIC/SCOM4PAD2/TC5, J28.3
- new net N$10: D5.A, R5.1
- new net N$3: IC1.PA13/I2C/EIC/SCOM2PAD1+/TC2
- new net N$4: D1.C, R1.2
- new net N$5: D2.C, R2.2
- new net N$6: R3.1, U1.EN
- new net N$8: D4.C, R4.2
- new net RDX: IC1.PB23/EIC/SCOM5PAD3
- new net RX_LED: IC1.PB3/EIC/AIN11/SCOM5PAD1, R1.1
- new net SCK: IC1.PB11/EIC/SCOM4PAD3/TC5, J28.4
- new net SCL: IC1.PA23/I2C/EIC/SCOM5PAD1+/TC4, J1.2
- new net SDA: IC1.PA22/I2C/EIC/SCOM5PAD0+/TC4, J1.1
- new net TDX: IC1.PB22/EIC/SCOM5PAD2
- new net TX_LED: IC1.PA27/EIC, R2.1
- new net USBHOSTEN: IC1.PA28/EIC
- new net VBAT: D3.A, J21.+
- net +3V3: now also C8.2, D1.A, D2.A, D4.A, IC1.VDDANA, J28.14, J28.5, J3.4, J4.4; no longer C3.2, C4.1, R2.2
- net D10: now also J1.13
- net D11: now also J1.14
- net D12: now also J1.15
- net D13: now also J3.1, R5.2
- net D2: now also J1.5
- net D3: now also J1.6
- net D4: now also J1.7
- net D5: now also J1.8
- net D6: now also J1.9
- net D7: now also J1.10
- net D8: now also J1.11
- net D9: now also J1.12
- net GND: now also C10.1, C9.1, D5.C, J21.-, J28.1, J28.12, J3.2, J4.1, J4.2, R4.1; no longer C3.1, C4.2
- net RESET: now also IC1.RESETN, J28.15; no longer R1.2, R2.1
- net VBUS: now also C10.2, D3.C, R3.2, U1.IN
Other:
- moved on the sheet: C5, C7, C8, R1, R2, S1, U1
